File: electronics/N80NA01/PROBE_V.kicad_sch (KiCad schematic)
At the start: 31 parts, among them Q10 2SA495G-0, Q11 2SC372G-0, Q12 2SA495G-0, Q13 2SC484-Y, Q14 2SA484-Y, Q15 2SA484-Y, Q16 2SC484-Y, Q9 2SC372G-0, U4 LM741

Commit message: Updated the probe driver schematics
Parts:
- added J1: Conn_01x01_Pin, symbol Connector:Conn_01x01_Pin
- added N80N07_R23, N80N07_R24: 1k, symbol Device:R_Small
- added N80N07_R25, N80N07_R26: 510R, symbol Device:R_Small
- added N80N07_R27: 300R, symbol Device:R_Small
- added N80N07_R28, N80N07_R29: 200R, symbol Device:R_Small
- added N80N07_R3, N80N07_R4: 2R, symbol Device:R
- added N80N07_R30, N80N07_R31: 100R, symbol Device:R_Small
- added N80N07_R32, N80N07_R33: 30R, symbol Device:R_Small
- added N80N07_R34: 20R, symbol Device:R_Small
- added N80N07_R35: 10R, symbol Device:R_Small
- added N80N07_R36: 5.1R, symbol Device:R_Small
- added N80N07_R37: 2R, symbol Device:R_Small
- added N80N07_R38: 3R, symbol Device:R
- added N80N07_R6: 20R, symbol Device:R
- added N80N07_S1-2: MAGNIFICATION, symbol Connector:Conn_01x16_Socket
- added N80N07_TR3: 2SD-110-0, symbol Device:Q_NPN
- added N80N07_TR4: 2SA663-Y, symbol Device:Q_PNP
- added SCAN_COIL_V: L, symbol Device:L
Connections:
- net +18V: now also N80N07_TR3.C
- net -18V: now also N80N07_TR4.C
- net PIN20: now also N80N07_TR4.B
- net PINX: now also N80N07_TR3.B
- net NF(V) renamed MAG_SWITCH(V)
- net MAG_SWITCH(V): now also J1.1 (Pin_1)
- new net: N80N07_R3.2, N80N07_R4.1, N80N07_R6.1, SCAN_COIL_V.1
- new net: N80N07_R4.2, N80N07_TR4.E
- new net: N80N07_R3.1, N80N07_TR3.E
- new net: N80N07_R25.1, N80N07_R26.2, N80N07_S1-2.13 (Pin_13)
- new net: N80N07_R24.1, N80N07_R25.2, N80N07_S1-2.14 (Pin_14)
- new net: N80N07_R26.1, N80N07_R27.2, N80N07_S1-2.12 (Pin_12)
- new net: N80N07_R27.1, N80N07_R28.2, N80N07_S1-2.11 (Pin_11)
- new net: N80N07_R36.1, N80N07_R37.2, N80N07_S1-2.2 (Pin_2)
- new net: N80N07_R35.1, N80N07_R36.2, N80N07_S1-2.3 (Pin_3)
- new net: N80N07_R32.1, N80N07_R33.2, N80N07_S1-2.6 (Pin_6)
- new net: N80N07_R31.1, N80N07_R32.2, N80N07_S1-2.7 (Pin_7)
- new net: N80N07_R37.1, N80N07_R38.1, N80N07_S1-2.1 (Pin_1)
- new net: N80N07_R23.1, N80N07_R24.2, N80N07_S1-2.15 (Pin_15)
- new net: N80N07_R23.2, N80N07_R6.2, N80N07_S1-2.16 (Pin_16), SCAN_COIL_V.2
- new net: N80N07_R30.1, N80N07_R31.2, N80N07_S1-2.8 (Pin_8)
- new net: N80N07_R29.1, N80N07_R30.2, N80N07_S1-2.9 (Pin_9)
- new net: N80N07_R33.1, N80N07_R34.2, N80N07_S1-2.5 (Pin_5)
- new net: N80N07_R28.1, N80N07_R29.2, N80N07_S1-2.10 (Pin_10)
- new net: N80N07_R34.1, N80N07_R35.2, N80N07_S1-2.4 (Pin_4)
- new net E(H): N80N07_R38.2
Other:
- note added: "Electron Column"
- note added: "N80N07"
- moved on the sheet: C15, C16, C30, Q10, Q11, Q12, Q13, Q14, Q15, Q16, Q9, R12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
