File: electronics/N80HD01/15V_regulated_supply/15V_regulated_supply.kicad_sch (KiCad schematic)
At the start: 35 parts, among them IC3 LM741, IC4 LM741

Commit message: Update front page
Parts:
- Rload3: value 100 -> 1k
Changed lines of the file:
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@@
 			)
 		)
-		(property "Value" "100"
+		(property "Value" "1k"
 			(at 217.17 92.7099 0)
 			(effects
